File: hardware/hardware.kicad_pcb (KiCad board)
At the start: 0 parts

Commit message: Completed all sircuit diagram and pcb design
Parts:
- added 3.7V1: Battery, Battery:BatteryHolder_Bulgin_BX0123_1xCR123, F.Cu at (40.7, 75.5)
- added BZ1: Buzzer, Buzzer_Beeper:Buzzer_12x9.5RM7.6, F.Cu at (107.2, 70.0)
- added D1: LED, LED_THT:LED_D10.0mm, F.Cu at (77.5, 164.5)
- added D2: LED, LED_THT:LED_D10.0mm, F.Cu at (77.0, 149.5)
- added D3: LED, LED_THT:LED_D10.0mm, F.Cu at (77.0, 134.5)
- added M1: Motor_DC, Motors:Vybronics_VZ30C1T8219732L, F.Cu at (116.7, 166.0)
- added Q1: 2N2219, Package_TO_SOT_THT:TO-92L_HandSolder, F.Cu at (95.5, 127.0)
- added Q2: 2N2219, Package_TO_SOT_THT:TO-92L_HandSolder, F.Cu at (95.0, 142.0)
- added Q3: 2N2219, Package_TO_SOT_THT:TO-92L_HandSolder, F.Cu at (95.5, 156.8)
- added Q4: Q_NPN_Darlington_BCEC, Package_TO_SOT_THT:TO-92L_HandSolder, F.Cu at (112.8, 84.5)
- added Q5: 2N2219, Package_TO_SOT_THT:TO-92L_HandSolder, F.Cu at (111.8, 93.8)
- added R1: 220R, Resistor_THT:R_Axial_DIN0207_L6.3mm_D2.5mm_P15.24mm_Horizontal, F.Cu at (89.3, 135.0)
- added R2: 220R, Resistor_THT:R_Axial_DIN0207_L6.3mm_D2.5mm_P15.24mm_Horizontal, F.Cu at (89.9, 148.5)
- added R3: 1K, Resistor_THT:R_Axial_DIN0207_L6.3mm_D2.5mm_P15.24mm_Horizontal, F.Cu at (90.4, 166.0)
- added R4: 1K, Resistor_THT:R_Axial_DIN0207_L6.3mm_D2.5mm_P15.24mm_Horizontal, F.Cu at (105.5, 94.1)
- added R5: 1K, Resistor_THT:R_Axial_DIN0207_L6.3mm_D2.5mm_P15.24mm_Horizontal, F.Cu at (110.5, 123.1)
- added R6: 220R, Resistor_THT:R_Axial_DIN0207_L6.3mm_D2.5mm_P15.24mm_Horizontal, F.Cu at (110.5, 141.6)
- added R7: 1K, Resistor_THT:R_Axial_DIN0207_L6.3mm_D2.5mm_P15.24mm_Horizontal, F.Cu at (110.5, 161.1)
- added R8: 1K, Resistor_THT:R_Axial_DIN0207_L6.3mm_D2.5mm_P15.24mm_Horizontal, F.Cu at (85.4, 86.5)
- added R9: 220R, Resistor_THT:R_Axial_DIN0207_L6.3mm_D2.5mm_P15.24mm_Horizontal, F.Cu at (85.9, 92.5)
- added SW1: SW_SPST, Button_Switch_THT:SW_Push_2P1T_Toggle_CK_PVA1xxH4xxxxxxV2, F.Cu at (92.5, 72.5)
- added U1: A4954, Package_SO:TSSOP-16-1EP_4.4x5mm_P0.65mm_EP3x3mm, F.Cu at (42.4, 97.6)
- added U2: TMP100, Package_TO_SOT_SMD:SOT-23-6, F.Cu at (41.4, 115.0)
- added U4: MPU-6050, Sensor_Motion:InvenSense_QFN-24_4x4mm_P0.5mm, F.Cu at (53.8, 115.0)
- added U5: MAX30102, OptoDevice:Maxim_OLGA-14_3.3x5.6mm_P0.8mm, F.Cu at (63.3, 97.8)
- added U6: ESP32-S2-WROVER, RF_Module:ESP32-C3-DevKitM-1, F.Cu at (43.1, 135.5)
- added U7: CN3158, Package_SO:SOIC-8-1EP_3.9x4.9mm_P1.27mm_EP2.41x3.3mm_ThermalVias, F.Cu at (52.6, 97.6)
Other:
- board outline added: 84.5 x 111 mm
- copper layers 0 -> 2
