File: hardware/hardware.kicad_sch (KiCad schematic)
At the start: 28 parts, among them M1 Motor_DC, M2 Stepper_Motor_unipolar_5pin, Q1 2N2219, Q2 2N2219, Q3 2N2219, Q4 Q_NPN_Darlington_BCEC, Q5 2N2219, SW1 SW_SPST, U1 A4954, U2 TMP100, U4 MPU-6050, U5 MAX30102, U6 ESP32-S2-WROVER, U7 CN3158

Commit message: Completed all sircuit diagram and pcb design
Parts:
- 3.7V1: footprint (none) -> Battery:BatteryHolder_Bulgin_BX0123_1xCR123
- BZ1: footprint (none) -> Buzzer_Beeper:Buzzer_12x9.5RM7.6
- D1, D2, D3: footprint (none) -> LED_THT:LED_D10.0mm
- M1: footprint (none) -> Motors:Vybronics_VZ30C1T8219732L
- Q1, Q2, Q3, Q5: footprint Package_TO_SOT_THT:TO-39-3 -> Package_TO_SOT_THT:TO-92L_HandSolder
- Q4: footprint (none) -> Package_TO_SOT_THT:TO-92L_HandSolder
- R1, R2, R3, R4, R5, R6, R7, R8, R9: footprint (none) -> Resistor_THT:R_Axial_DIN0207_L6.3mm_D2.5mm_P15.24mm_Horizontal
- SW1: footprint (none) -> Button_Switch_THT:SW_Push_2P1T_Toggle_CK_PVA1xxH4xxxxxxV2
- U6: footprint RF_Module:ESP32-S2-WROVER -> RF_Module:ESP32-C3-DevKitM-1
Changed lines of the file:
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@@
 		(company "DEPARTMENT OF COMPUTER ENGINEERING, UNILAG")
 		(comment 1 "190408063")
-		(comment 2 "Sinmi")
+		(comment 2 "Obafemi-Moses Mosinmiloluwa")
 	)
 	(rectangle
@@
 			)
 		)
-		(property "Footprint" ""
+		(property "Footprint" "Package_TO_SOT_THT:TO-92L_HandSolder"
 			(at 191.77 63.5 0)
 			(hide yes)
@@
 			)
 		)
-		(property "Footprint" ""
+		(property "Footprint" "LED_THT:LED_D10.0mm"
 			(at 195.58 93.98 0)
 			(hide yes)
@@
 			)
 		)
-		(property "Footprint" ""
+		(property "Footprint" "Button_Switch_THT:SW_Push_2P1T_Toggle_CK_PVA1xxH4xxxxxxV2"
 			(at 78.74 110.49 0)
 			(hide yes)
@@
 			)
 		)
-		(property "Footprint" ""
+		(property "Footprint" "LED_THT:LED_D10.0mm"
 			(at 233.68 74.93 0)
 			(hide yes)
@@
 			)
 		)
-		(property "Footprint" ""
+		(property "Footprint" "Resistor_THT:R_Axial_DIN0207_L6.3mm_D2.5mm_P15.24mm_Horizontal"
 			(at 230.378 58.42 90)
 			(hide yes)
@@
 			)
 		)
-		(property "Footprint" ""
+		(property "Footprint" "Resistor_THT:R_Axial_DIN0207_L6.3mm_D2.5mm_P15.24mm_Horizontal"
 			(at 214.63 48.768 90)
 			(hide yes)
@@
 			)
 		)
-		(property "Footprint" ""
+		(property "Footprint" "Buzzer_Beeper:Buzzer_12x9.5RM7.6"
 			(at 230.505 33.02 90)
 			(hide yes)
@@
 			)
 		)
-		(property "Footprint" ""
+		(property "Footprint" "Battery:BatteryHolder_Bulgin_BX0123_1xCR123"
 			(at 49.53 121.666 90)
 			(hide yes)
@@
 			)
 		)
-		(property "Footprint" "RF_Module:ESP32-S2-WROVER"
+		(property "Footprint" "RF_Module:ESP32-C3-DevKitM-1"
 			(at 170.18 110.49 0)
 			(hide yes)
@@
 			)
 		)
-		(property "Footprint" "Package_TO_SOT_THT:TO-39-3"
+		(property "Footprint" "Package_TO_SOT_THT:TO-92L_HandSolder"
 			(at 233.68 122.555 0)
 			(hide yes)
@@
 			)
 		)
-		(property "Footprint" ""
+		(property "Footprint" "Resistor_THT:R_Axial_DIN0207_L6.3mm_D2.5mm_P15.24mm_Horizontal"
 			(at 229.362 132.08 90)
 			(hide yes)
@@
 			)
 		)
-		(property "Footprint" ""
+		(property "Footprint" "Resistor_THT:R_Axial_DIN0207_L6.3mm_D2.5mm_P15.24mm_Horizontal"
 			(at 231.902 95.25 90)
 			(hide yes)
@@
 			)
 		)
-		(property "Footprint" "Package_TO_SOT_THT:TO-39-3"
+		(property "Footprint" "Package_TO_SOT_THT:TO-92L_HandSolder"
 			(at 198.12 107.315 0)
 			(hide yes)
@@
 			)
 		)
-		(property "Footprint" "Package_TO_SOT_THT:TO-39-3"
+		(property "Footprint" "Package_TO_SOT_THT:TO-92L_HandSolder"
 			(at 231.14 48.895 0)
 			(hide yes)
@@
 			)
 		)
-		(property "Footprint" ""
+		(property "Footprint" "Resistor_THT:R_Axial_DIN0207_L6.3mm_D2.5mm_P15.24mm_Horizontal"
 			(at 177.8 67.818 90)
 			(hide yes)
@@
 			)
 		)
-		(property "Footprint" ""
+		(property "Footprint" "Resistor_THT:R_Axial_DIN0207_L6.3mm_D2.5mm_P15.24mm_Horizontal"
 			(at 220.98 85.598 90)
 			(hide yes)
@@
 			)
 		)
-		(property "Footprint" ""
+		(property "Footprint" "LED_THT:LED_D10.0mm"
 			(at 231.14 109.22 0)
 			(hide yes)
@@
 			)
 		)
-		(property "Footprint" ""
+		(property "Footprint" "Resistor_THT:R_Axial_DIN0207_L6.3mm_D2.5mm_P15.24mm_Horizontal"
 			(at 181.61 107.188 90)
 			(hide yes)
@@
 			)
 		)
-		(property "Footprint" ""
+		(property "Footprint" "Resistor_THT:R_Axial_DIN0207_L6.3mm_D2.5mm_P15.24mm_Horizontal"
 			(at 193.802 116.84 90)
 			(hide yes)
@@
 			)
 		)
-		(property "Footprint" ""
+		(property "Footprint" "Motors:Vybronics_VZ30C1T8219732L"
 			(at 190.5 49.276 0)
 			(hide yes)
@@
 			)
 		)
-		(property "Footprint" ""
+		(property "Footprint" "Resistor_THT:R_Axial_DIN0207_L6.3mm_D2.5mm_P15.24mm_Horizontal"
 			(at 217.17 122.428 90)
 			(hide yes)
@@
 			)
 		)
-		(property "Footprint" "Package_TO_SOT_THT:TO-39-3"
+		(property "Footprint" "Package_TO_SOT_THT:TO-92L_HandSolder"
 			(at 236.22 85.725 0)
 			(hide yes)
